File: phasefreq.kicad_pcb (KiCad board)
At the start: 4 copper layers, 90.5 x 56 mm, 113 parts, among them J1 Power Input, J2 RF Input, J3 LO Input, J4 VCO Tune, U1 LM317_3PinPackage, U2 LM337_SOT223, U3 ADCMP564, U4 AD9901, U5 LM4040DIZ-2.5, U6 AD8676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

Commit message: add thermal pads for regulators, increment to revB2
Parts:
- moved C7 32.4 mm to (131.2, 94.2), turned to 90 degrees
- moved C6 12.9 mm to (146.2, 94.3), turned to 270 degrees
- moved C4 7.75 mm to (142.5, 95.0)
- moved C1 7.25 mm to (135.0, 95.0)
- moved J1 5.10 mm to (141.2, 86.0), turned to 180 degrees
- moved U2 2.02 mm to (163.2, 87.5)
- moved U1 0.56 mm to (150.8, 87.5)
Routing:
- net Net-(C1-Pad2): track 32.7 -> 41.7 mm, vias 0 -> 14
- net Net-(C4-Pad1): track 25.2 -> 18.7 mm
- net GNDA: track 288.2 -> 291.4 mm, vias 150 -> 148
- net Net-(FB2-Pad2): track 7.77 -> 8.45 mm
- net Net-(R3-Pad2): track 17.2 -> 17.3 mm, vias 2 -> 5
- net Net-(FB1-Pad1): track 8.93 -> 9.03 mm, vias 0 -> 7
- added copper zone on B.Cu, net Net-(C1-Pad2)
- added copper zone on F.Cu, net Net-(C1-Pad2)
- added copper zone on B.Cu, net Net-(FB1-Pad1)
- added copper zone on F.Cu, net Net-(FB1-Pad1)
Other:
- board text added: "revB2 2019-02 @rwpeterson"
- board text removed: "revB1 Dec 2019 @rwpeterson"
